File: Q917/Q917.kicad_sch (KiCad schematic)
At the start: 26 parts, among them J1 Analog, J10 SELE, J11 RESET, J2 Digital, J3 to_W5500, J4 to_LCD, J5 to_TEMP, J6 to_HUMI, J7 to_ILLU, J8 to_ETC, J9 DC5V, P10 SELE_SW, P11 RESET_SW, P5 TEMP_POT, P6 HUMI_POT, P7 ILLUMI_POT, P8 ETC_POT, SW1 RESET, SW2 SELE

Commit message: UNO版はじめ
Parts:
- removed C1: 100uF/25V, symbol Device:C_Polarized_Small
- removed J1: Analog, Connector_PinSocket_2.54mm:PinSocket_1x15_P2.54mm_Vertical, symbol Connector_Generic:Conn_01x15
- removed J2: Digital, Connector_PinSocket_2.54mm:PinSocket_1x15_P2.54mm_Vertical, symbol Connector_Generic:Conn_01x15
- removed J9: DC5V, Connector_BarrelJack:BarrelJack_Horizontal, symbol Connector:Jack-DC
- removed R1, R2: 10k, Resistor_THT:R_Axial_DIN0204_L3.6mm_D1.6mm_P7.62mm_Horizontal, symbol Device:R_US
- added A1: Arduino_UNO_R3, Module:Arduino_UNO_R3, symbol MCU_Module:Arduino_UNO_R3
- J5: value to_TEMP -> to_VR1
- J6: value to_HUMI -> to_VR2
- J7: value to_ILLU -> to_VR3
- J8: value to_ETC -> to_VR4
Connections:
- net A0: now also A1.9 (A0)
- net A1: now also A1.10 (A1)
- net A2: now also A1.11 (A2)
- net A3: now also A1.12 (A3)
- net A4/SDA: now also A1.31 (SDA/A4)
- net A5/SCL: now also A1.32 (SCL/A5)
- net D13/SCK: now also A1.28 (D13)
- net GND: now also J11.1 (Pin_1); no longer J11.2 (Pin_2)
- net ~{RESET}: now also J11.2 (Pin_2), A1.3 (~{RESET}); no longer J11.1 (Pin_1)
- net *D10/SS: no longer names the net of J3.4 (Pin_4)
- net *D10/SS: now also A1.25 (D10)
- net *D11/MOSI: no longer names the net of J3.6 (Pin_6)
- net *D11/MOSI: now also A1.26 (D11)
- net *D9: no longer names the net of J10.1 (Pin_1)
- net *D9: now also A1.24 (D9)
- net D12/MISO: no longer names the net of J3.8 (Pin_8)
- net D12/MISO: now also A1.27 (D12)
- no-connect marks 14 -> 11
Other:
- title: UECS Simulator for DEN-NOH-01 -> UECS Simulator Q917B
- moved on the sheet: J10, J11, J4, J5, J6, J7, J8

Commit message: 回路変更
Parts:
- added J1: AUTO, Connector_JST:JST_XH_B2B-XH-A_1x02_P2.50mm_Vertical, symbol Connector_Generic:Conn_01x02
- added J12: SW4, Connector_JST:JST_XH_B2B-XH-A_1x02_P2.50mm_Vertical, symbol Connector_Generic:Conn_01x02
- added J13: SW3, Connector_JST:JST_XH_B2B-XH-A_1x02_P2.50mm_Vertical, symbol Connector_Generic:Conn_01x02
- added J2: SW2, Connector_JST:JST_XH_B2B-XH-A_1x02_P2.50mm_Vertical, symbol Connector_Generic:Conn_01x02
- added J9: SW1, Connector_JST:JST_XH_B2B-XH-A_1x02_P2.50mm_Vertical, symbol Connector_Generic:Conn_01x02
- added P1: SW1, symbol Connector:Conn_01x02_Male
- added P2: SW2, symbol Connector:Conn_01x02_Male
- added P3: SW4, symbol Connector:Conn_01x02_Male
- added P4: SW3, symbol Connector:Conn_01x02_Male
- added SW3: SW1, symbol Switch:SW_Push
- added SW4: SW2, symbol Switch:SW_Push
- added SW5: SW4, symbol Switch:SW_Push
- added SW6: SW3, symbol Switch:SW_Push
Connections:
- net GND: now also A1.29 (GND), A1.6 (GND), A1.7 (GND), J1.2 (Pin_2), J12.2 (Pin_2), J13.2 (Pin_2), J2.2 (Pin_2), J9.2 (Pin_2)
- net at A1.17 (D2): now also J10.1 (Pin_1)
- net at A1.18 (D3): now also J1.1 (Pin_1)
- net at A1.19 (D4): now also J9.1 (Pin_1)
- net at A1.20 (D5): now also J2.1 (Pin_1)
- net at A1.21 (D6): now also J13.1 (Pin_1)
- net at A1.22 (D7): now also J12.1 (Pin_1)
- net at A1.24 (D9): no longer J10.1 (Pin_1)
- new net: P2.1 (Pin_1), SW4.1
- new net: P2.2 (Pin_2), SW4.2
- new net: P3.1 (Pin_1), SW5.1
- new net: P3.2 (Pin_2), SW5.2
- new net: P4.1 (Pin_1), SW6.1
- new net: P4.2 (Pin_2), SW6.2
- new net: P1.1 (Pin_1), SW3.1
- new net: P1.2 (Pin_2), SW3.2
- no-connect marks 11 -> 9
Other:
- moved on the sheet: J10, P10, P11, SW1, SW2
